File: kicad/solder-reflow.kicad_pcb (KiCad board)
At the start: 2 copper layers, 109.3 x 100.5 mm, 39 parts, among them J1 XT60PW-M, J2 1985807, J3 Conn_01x06_Male, U1 ESP32-WROOM-32E-N8, U2 DGD0215WT-7, U3 AP62201WU-7, U4 MAX31855KASA+T

Commit message: Tweaked layout; refined buck layout; added graphics
Parts:
- added G***: LOGO, footprint:OSH9mm, B.Cu at (64.1, 38.0)
- G***: footprint graphic footprints:IdeaUpLogoText7mm -> footprint:IdeaUpLogoText7mm
- moved C2 4.77 mm to (56.4, 42.7), turned to -90 degrees
- moved C4 3.78 mm to (60.6, 44.8), turned to 90 degrees
- moved J2 3.47 mm to (99.1, 59.5), turned to 180 degrees
- moved C5 2.82 mm to (67.3, 42.7)
- moved R6 2.23 mm to (67.3, 46.1)
- moved L1 1.90 mm to (62.9, 39.1)
- moved C1 1.66 mm to (58.4, 42.7), turned to -90 degrees
- moved R7 1.01 mm to (65.0, 47.3), turned to 180 degrees
- moved U3 0.88 mm to (64.2, 44.4)
Connections:
- J2 pad 1: TC- -> TC+
- J2 pad 2: TC+ -> TC-
Routing:
- net +3V3: track 182.8 -> 166.5 mm
- net Net-(C5-Pad1): track 10.2 -> 0.00 mm
- net HEATER: track 2945.9 -> 2948.4 mm, vias 11 -> 8
- net Net-(C5-Pad2): track 2.77 -> 1.81 mm
- net GND: vias 224 -> 242
- added copper zone on F.Cu, net +3V3
- added copper zone on F.Cu, net Net-(C5-Pad1)
Other:
- board text added: "WIFI RESET"
- board text added: "github.com/ideaup-online/esp32-reflow-plate"
- board text removed: "WiFi RESET"

Commit message: Changed tactile switch part
Parts:
- S1: value B3U-1000PM-B -> PTS810SJM250SMTRLFS; footprint mouser_ecad:B3U1000PMB -> mouser_ecad:PTS810SJG250SMTRLFS
- moved S1 0.27 mm to (129.1, 58.8)
Connections:
- S1 pad 1: GND -> GPIO0
Routing:
- net GPIO0: track 75.9 -> 79.1 mm
Changed lines of the file:
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@@
       ) (layer "F.SilkS") (width 0) (fill solid))
   )
-  (footprint "mouser_ecad:B3U1000PMB" (layer "F.Cu")
-    (at 129 59 90)
-    (descr "B3U-1000PM-B-2")
-    (tags "Switch")
-    (property "Description" "Microswitch TACT; SPST-NO; Pos:2; 0.05A/24VDC; SMT; 1.5N; 2.5x3mm")
-    (property "Height" "1.75")
-    (property "Manufacturer_Name" "Omron Electronics")
-    (property "Manufacturer_Part_Number" "B3U-1000PM-B")
-    (property "Mouser Part Number" "653-B3U-1000PM-B")
-    (property "Mouser Price/Stock" "https://www.mouser.co.uk/ProductDetail/Omron-Electronics/B3U-1000PM-B?qs=hnUcNC2tU0oErWp7o87bxg%3D%3D")
-    (property "Sheetfile" "solder-reflow.kicad_sch")
-    (property "Sheetname" "")
-    (attr through_hole)
-    (fp_text reference "S1" (at 0.55 0 90) (layer "F.Fab")
-      (effects (font (size 1.27 1.27) (thickness 0.254)))
-    )
-    (fp_text value "B3U-1000PM-B" (at 0.55 0 90) (layer "F.SilkS") hide
-      (effects (font (size 1.27 1.27) (thickness 0.254)))
-    )
-    (fp_text user "${REFERENCE}" (at 0.55 0 90) (layer "F.Fab")
-      (effects (font (size 1.27 1.27) (thickness 0.254)))
-    )
-    (fp_line (start 1.5 -1.25) (end -1.5 -1.25) (layer "F.SilkS") (width 0.1))
-    (fp_line (start 3.2 0) (end 3.2 0) (layer "F.SilkS") (width 0.1))
-    (fp_line (start 3.1 0) (end 3.1 0) (layer "F.SilkS") (width 0.1))
-    (fp_line (start 1.5 1.25) (end -1.5 1.25) (layer "F.SilkS") (width 0.1))
-    (fp_arc (start 3.2 0) (mid 3.15 0.05) (end 3.1 0) (layer "F.SilkS") (width 0.1))
-    (fp_arc (start 3.1 0) (mid 3.15 -0.05) (end 3.2 0) (layer "F.SilkS") (width 0.1))
-    (fp_line (start 4.2 -2.25) (end 4.2 2.25) (layer "F.CrtYd") (width 0.1))
-    (fp_line (start -3.1 2.25) (end -3.1 -2.25) (layer "F.CrtYd") (width 0.1))
-    (fp_line (start 4.2 2.25) (end -3.1 2.25) (layer "F.CrtYd") (width 0.1))
-    (fp_line (start -3.1 -2.25) (end 4.2 -2.25) (layer "F.CrtYd") (width 0.1))
-    (fp_line (start -1.5 -1.25) (end -1.5 1.25) (layer "F.Fab") (width 0.2))
-    (fp_line (start 1.5 -1.25) (end -1.5 -1.25) (layer "F.Fab") (width 0.2))
-    (fp_line (start -1.5 1.25) (end 1.5 1.25) (layer "F.Fab") (width 0.2))
-    (fp_line (start 1.5 1.25) (end 1.5 -1.25) (layer "F.Fab") (width 0.2))
-    (pad "" np_thru_hole circle locked (at 0 0 90) (size 0.85 0.85) (drill 0.85) (layers *.Cu *.Mask))
-    (pad "1" smd rect locked (at 1.7 0 90) (size 0.8 1.7) (layers "F.Cu" "F.Paste" "F.Mask")
-      (net 1 "GND") (pinfunction "COM") (pintype "passive"))
-    (pad "2" smd rect locked (at -1.7 0 90) (size 0.8 1.7) (layers "F.Cu" "F.Paste" "F.Mask")
-      (net 28 "GPIO0") (pinfunction "NO") (pintype "passive"))
-    (model "B3U-1000PM-B.stp"
-      (offset (xyz 0 0 0))
-      (scale (xyz 1 1 1))
-      (rotate (xyz 0 0 0))
-    )
-  )
   (footprint "digikey-footprints:0603" (layer "F.Cu")
     (at 67.3 46.1 90)
@@
       (net 28 "GPIO0") (pintype "passive"))
   )
-  (footprint "digikey-footprints:0603" (layer "F.Cu")
+  (footprint "digikey-footprints:0603" locked (layer "F.Cu")
     (at 125 59 90)
     (property "Sheetfile" "solder-reflow.kicad_sch")
@@
     )
   )
+  (footprint "mouser_ecad:PTS810SJG250SMTRLFS" (layer "F.Cu")
+    (at 129.1 58.75 90)
+    (descr "pts810")
+    (tags "Switch")
+    (property "Description" "PTS810SJM250SMTRLFS (Tactile Switches)")
+    (property "Height" "")
+    (property "Manufacturer_Name" "C & K COMPONENTS")
+    (property "Manufacturer_Part_Number" "PTS810SJM250SMTRLFS")
+    (property "Mouser Part Number" "611-PTS810SJM250SMTR")
+    (property "Mouser Price/Stock" "https://www.mouser.co.uk/ProductDetail/CK/PTS810SJM250SMTRLFS?qs=UxeAxwACbqnyNdXLIf%2FqnQ%3D%3D")
+    (property "Sheetfile" "solder-reflow.kicad_sch")
+    (property "Sheetname" "")
+    (attr smd)
+    (fp_text reference "S1" (at 0.025 0 180) (layer "F.SilkS")
+      (effects (font (size 1 1) (thickness 0.15)))
+    )
+    (fp_text value "PTS810SJM250SMTRLFS" (at -0.25 0 90) (layer "F.SilkS") hide
+      (effects (font (size 1.27 1.27) (thickness 0.254)))
+    )
+    (fp_text user "${REFERENCE}" (at -0.25 0 90) (layer "F.Fab")
+      (effects (font (size 1.27 1.27) (thickness 0.254)))
+    )
+    (fp_line (start -2.1 -1.6) (end 2.075 -1.6) (layer "F.SilkS") (width 0.1))
+    (fp_line (start -3 -1) (end -3 -1) (layer "F.SilkS") (width 0.2))
+    (fp_line (start -2.1 1.6) (end 2.075 1.6) (layer "F.SilkS") (width 0.1))
+    (fp_line (start -3 -1.2) (end -3 -1.2) (layer "F.SilkS") (width 0.2))
+    (fp_arc (start -3 -1.2) (mid -2.9 -1.1) (end -3 -1) (layer "F.SilkS") (width 0.2))
+    (fp_arc (start -3 -1) (mid -3.1 -1.1) (end -3 -1.2) (layer "F.SilkS") (width 0.2))
+    (fp_line (start 3.6 2.6) (end -4.1 2.6) (layer "F.CrtYd") (width 0.1))
+    (fp_line (start -4.1 2.6) (end -4.1 -2.6) (layer "F.CrtYd") (width 0.1))
+    (fp_line (start -4.1 -2.6) (end 3.6 -2.6) (layer "F.CrtYd") (width 0.1))
+    (fp_line (start 3.6 -2.6) (end 3.6 2.6) (layer "F.CrtYd") (width 0.1))
+    (fp_line (start -2.1 -1.6) (end 2.1 -1.6) (layer "F.Fab") (width 0.2))
+    (fp_line (start -2.1 1.6) (end -2.1 -1.6) (layer "F.Fab") (width 0.2))
+    (fp_line (start 2.1 1.6) (end -2.1 1.6) (layer "F.Fab") (width 0.2))
+    (fp_line (start 2.1 -1.6) (end 2.1 1.6) (layer "F.Fab") (width 0.2))
+    (pad "1" smd rect locked (at -2.075 -1.075 180) (size 0.65 1.05) (layers "F.Cu" "F.Paste" "F.Mask")
+      (net 28 "GPIO0") (pinfunction "1") (pintype "passive"))
+    (pad "2" smd rect locked (at 2.075 -1.075 180) (size 0.65 1.05) (layers "F.Cu" "F.Paste" "F.Mask")
+      (net 28 "GPIO0") (pinfunction "2") (pintype "passive"))
+    (pad "3" smd rect locked (at -2.075 1.075 180) (size 0.65 1.05) (layers "F.Cu" "F.Paste" "F.Mask")
+      (net 1 "GND") (pinfunction "3") (pintype "passive"))
+    (pad "4" smd rect locked (at 2.075 1.075 180) (size 0.65 1.05) (layers "F.Cu" "F.Paste" "F.Mask")
+      (net 1 "GND") (pinfunction "4") (pintype "passive"))
+  )
   (footprint "digikey-footprints:0603" locked (layer "F.Cu")
     (at 115 60 90)
@@
   (via (at 136.36 55.14) (size 0.8) (drill 0.4) (layers "F.Cu" "B.Cu") (free) (net 1))
   (via (at 110.96 44.98) (size 0.8) (drill 0.4) (layers "F.Cu" "B.Cu") (free) (net 1))
-  (via (at 131.28 57.68) (size 0.8) (drill 0.4) (layers "F.Cu" "B.Cu") (free) (net 1))
+  (via (at 131.3 56.675) (size 0.8) (drill 0.4) (layers "F.Cu" "B.Cu") (free) (net 1))
   (via (at 101.9 57.5) (size 0.8) (drill 0.4) (layers "F.Cu" "B.Cu") (free) (net 1))
   (via (at 133.82 52.6) (size 0.8) (drill 0.4) (layers "F.Cu" "B.Cu") (free) (net 1))
@@
   (via (at 47.84 47.52) (size 0.8) (drill 0.4) (layers "F.Cu" "B.Cu") (free) (net 1))
   (via (at 35.14 55.14) (size 0.8) (drill 0.4) (layers "F.Cu" "B.Cu") (free) (net 1))
-  (via (at 131.28 61) (size 0.8) (drill 0.4) (layers "F.Cu" "B.Cu") (free) (net 1))
+  (via (at 131.3 60.825) (size 0.8) (drill 0.4) (layers "F.Cu" "B.Cu") (free) (net 1))
   (via (at 123.66 42.44) (size 0.8) (drill 0.4) (layers "F.Cu" "B.Cu") (free) (net 1))
   (via (at 61.5 56.3) (size 0.8) (drill 0.4) (layers "F.Cu" "B.Cu") (free) (net 1))
@@
   (segment (start 87.6 52.4) (end 95.385 44.615) (width 0.25) (layer "B.Cu") (net 15))
   (segment (start 120.6 62.8) (end 123 60.4) (width 0.25) (layer "F.Cu") (net 28))
-  (segment (start 127.3 60.7) (end 129 60.7) (width 0.25) (layer "F.Cu") (net 28))
   (segment (start 123 59.7) (end 125 59.7) (width 0.25) (layer "F.Cu") (net 28))
   (segment (start 89.207006 56.760178) (end 89.207006 59.207006) (width 0.25) (layer "F.Cu") (net 28))
+  (segment (start 128.025 60.825) (end 128.025 56.675) (width 0.25) (layer "F.Cu") (net 28))
+  (segment (start 125 59.7) (end 126.3 59.7) (width 0.25) (layer "F.Cu") (net 28))
+  (segment (start 127.425 60.825) (end 128.025 60.825) (width 0.25) (layer "F.Cu") (net 28))
   (segment (start 124 59.6) (end 124 51.65) (width 0.25) (layer "F.Cu") (net 28))
-  (segment (start 126.3 59.7) (end 127.3 60.7) (width 0.25) (layer "F.Cu") (net 28))
+  (segment (start 126.3 59.7) (end 127.425 60.825) (width 0.25) (layer "F.Cu") (net 28))
   (segment (start 92.8 62.8) (end 105.8 62.8) (width 0.25) (layer "F.Cu") (net 28))
   (segment (start 123 59.7) (end 123 60.4) (width 0.25) (layer "F.Cu") (net 28))
   (segment (start 89.207006 59.207006) (end 92.8 62.8) (width 0.25) (layer "F.Cu") (net 28))
   (segment (start 124 51.65) (end 108.35 36) (width 0.25) (layer "F.Cu") (net 28))
-  (segment (start 125 59.7) (end 126.3 59.7) (width 0.25) (layer "F.Cu") (net 28))
   (via (at 120.6 62.8) (size 0.8) (drill 0.4) (layers "F.Cu" "B.Cu") (net 28))
   (via (at 105.8 62.8) (size 0.8) (drill 0.4) (layers "F.Cu" "B.Cu") (net 28))
